Commit message: added_colors_robot

File: src/my_robot/urdf/my_robot.xacro (robot description, xacro)
@@ -30,7 +30,4 @@
         <box size=".4 .2 .1"/>
       </geometry>
-	<gazebo reference="chassis">
-  	  <material>Gazebo/Yellow</material>
-	</gazebo>
     </visual>
     <collision name='back_caster_collision'>
@@ -59,4 +56,13 @@
     </visual>
   </link>
+	<gazebo reference="chassis">
+          <material>Gazebo/Yellow</material>
+        </gazebo>
+	<gazebo reference="left_wheel">
+		<material>Gazebo/Blue</material>
+	</gazebo>
+	<gazebo reference="right_wheel">
+		<material>Gazebo/Blue</material>
+	</gazebo>
 	<!--Eriks code additions:-->
 	<link name= "left_wheel">
